File: minishirasu-firm/board/mini_shirasu.sch (EAGLE design)
At the start: 74 parts, among them CON1 XT30PW-F, IC2 LMR51606YDBVR, IC3 SN65HVD230DR, J1 SM02B-GHS-TB_LF__SN_, J5 EP2.5-4-SIDE, Q1 FH3406GS, Q2 FH3406GS, Q3 FH3406GS, Q4 FH3406GS, U11 INA2181A1IDGSR, U3 MPQ6528GVE-AEC1-ZQFN-28_MPQ65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, U7 STM32F302_303C2, U9 XC6206, Y1 X322512MSB4SI

Commit message: Update mini-shirasu board data to the 2025-12-02 revision
Replace the EAGLE schematic and board, and add the Gerber files
exported on 2025-12-02 under board/gerber/.

Co-Authored-By: Claude Opus 5.5 <noreply@anthropic.com>
Claude-Session: https://claude.ai/code/session_01XNr5i9z8ibucq78UtzMFbR
Parts:
- removed C33: 100n, Capacitor:C_CHIP-0402(1005-METRIC)
- removed IC2: LMR51606YDBVR, LMR51606YDBVR:LMR51606YDBVR
- removed IC3: SN65HVD230DR, SN65HVD230DR:SN65HVD230DR
- removed ISENSE, PWMB: TPB1,27, testpad:TPB1,27
- removed J1: SM02B-GHS-TB_LF__SN_, SM02B-GHS-TB_v2:SM02B-GHS-TB_LF__SN_
- removed R10: 100k, rcl:R-EU_R0402
- removed R13, R9: 5.1k, rcl:R-EU_R0402
- removed U3: MPQ6528GVE-AEC1-ZQFN-28_MPQ6528_MNP, MPQ6528GVE-AEC1-Z:MPQ6528GVE-AEC1-ZQFN-28_MPQ6528_MNP
- removed Y1: X322512MSB4SI, X322512MSB4SI:X322512MSB4SI
- added C31: 10u, rcl:C-EUC0805
- added C43, C44: 6800p, rcl:C-EUC0603
- added D1, D2: PMEG6010CEJ,115, nexperia:PMEG6010CEJ,115
- added IC1: DRV8701PRGER, DRV8701PRGER:DRV8701PRGER
- added J2: BM02B-GHS-TBT_LF__SN_, BM02B-GHS-TBT_LF__SN_:BM02B-GHS-TBT_LF__SN_
- added R14: 1k, rcl:R-EU_R0402
- added U1: XC9705B75CPR-GSOT-89-5_TOR-M, CRS_EAGLE_Lib:XC9705B75CPR-GSOT-89-5_TOR-M
- added U2: TJA1050T_CM,118, TJA1050T_CM_118:TJA1050T_CM,118
- added Y2: X50328MSB2GI, X50328MSB2GI:X50328MSB2GI
- C1, C11, C2, C28, C3: device Capacitor:C_CHIP-0402(1005-METRIC) -> rcl:C-EUC0402
- C10: value 1u25V -> 100n; device Capacitor:C_CHIP-0402(1005-METRIC) -> rcl:C-EUC0402
- C12: value 33p -> 1u25V; device Capacitor:C_CHIP-0402(1005-METRIC) -> rcl:C-EUC0402
- C13: value 33p -> 100n; device Capacitor:C_CHIP-0402(1005-METRIC) -> rcl:C-EUC0402
- C14: value 10u -> 10n; device rcl:C-EUC0805 -> rcl:C-EUC0402
- C15, C16: value 1u -> 1u25V; device rcl:C-EUC0603 -> rcl:C-EUC0402
- C17: value 470n -> 330p; device rcl:C-EUC0805 -> rcl:C-EUC0402
- C18: value 220u -> 330p; device Capacitor:C-POL_ECAP-10.5MM -> rcl:C-EUC0402
- C19: value 10u -> 100n; device rcl:C-EUC0805 -> rcl:C-EUC0402
- C21: value 6800p -> 10u; device rcl:C-EUC0603 -> rcl:C-EUC0805
- C22, C23: value 6800p -> 1u25V; device rcl:C-EUC0603 -> rcl:C-EUC0402
- C24: value 6800p -> 30p; device rcl:C-EUC0603 -> rcl:C-EUC0402
- C25: value 100n -> 6800p; device Capacitor:C_CHIP-0402(1005-METRIC) -> rcl:C-EUC0603
- C26: value 330p -> 6800p; device Capacitor:C_CHIP-0402(1005-METRIC) -> rcl:C-EUC0603
- C27: value 1u25V -> 30p; device Capacitor:C_CHIP-0402(1005-METRIC) -> rcl:C-EUC0402
- C29: value 100n -> 10u; device Capacitor:C_CHIP-0402(1005-METRIC) -> rcl:C-EUC0805
- C30: value 220u -> 10u; device Capacitor:C-POL_ECAP-10.5MM -> rcl:C-EUC0805
- C4: value 10n -> 100n; device Capacitor:C_CHIP-0402(1005-METRIC) -> rcl:C-EUC0402
- C5: value 1u25V -> 2.2u; device Capacitor:C_CHIP-0402(1005-METRIC) -> rcl:C-EUC0805
- C6: value 2.2u -> 22u
- C7: value 100n -> 22u; device Capacitor:C_CHIP-0402(1005-METRIC) -> rcl:C-EUC0805
- C8: value 100n -> 18p; device Capacitor:C_CHIP-0402(1005-METRIC) -> rcl:C-EUC0402
- C9: value 22u -> 1u; device rcl:C-EUC0805 -> rcl:C-EUC0603
- L1: value DFE252012F-100M=P2 -> 6.8u; device DFE252012F-100M=P2:DFE252012F-100M=P2 -> CRS_EAGLE_Lib:VLS252012CX-6R8M-1INDUCTOR_1008
- Q1, Q2, Q3, Q4: value FH3406GS -> BSZ042N06NSATMA1; device FH3406GS_PDFN5x6_8L:FH3406GS -> CRS_EAGLE_Lib:BSZ042N06NSATMA1
- R1: value 27k -> 120k
- R12: value 2m -> 1m
- R2: value 5.1k -> 680k; device rcl:R-EU_R0402 -> rcl:R-EU_R0603
- R5: value 5.1k -> 68k
- R6: value 27k -> 220k
- R7: value 1k -> 20k
- U11: MANUFACTURER_PART_NUMBER INA2181A2IDGSR -> (none)
- renumbered +5V to TP6, PWMA to TP8
Connections:
- removed net BST1: C16.1, U3.BSTA
- removed net BST2: C15.2, U3.BSTB
- removed net CB: C8.2, IC2.CB
- removed net CPA: C17.1, U3.CPA
- removed net CPB: C17.2, U3.CPB
- removed net DT: R5.2, U3.DT
- removed net N$2: C12.2, U7A.PF0-OSC_IN, Y1.CRYSTAL_1
- removed net N$3: C13.2, U7A.PF1-OSC_OUT, Y1.CRYSTAL_2
- removed net NSLEEP: U3.NSLEEP, U7A.PA2
- removed net OC_REF: R10.2, R13.1, U3.OC_REF
- removed net PWMA: TP8.TP, U3.PWMA, U7A.PA9
- removed net PWMB: PWMB.TP, U3.PWMB, U7A.PA8
- removed net SW: C8.1, IC2.SW, L1.2
- removed net VREG: C14.2, U3.VREG
- new net APWM: IC1.PH, U7A.PA9
- new net AVDD: C11.2, IC1.AVDD, R5.2, R6.2
- new net BPWM: IC1.EN, U7A.PA8
- new net CPH: C10.2, IC1.CPH
- new net CPL: C10.1, IC1.CPL
- new net DVDD: C12.2, IC1.DVDD
- new net IDRIVE: IC1.IDRIVE, R5.1
- new net ISENSEA: C18.2, R14.2, U7A.PA4
- new net LX: L1.1, U1.LX
- new net N$15: C24.2, U7A.PF0-OSC_IN, Y2.1
- new net N$20: C27.2, U7A.PF1-OSC_OUT, Y2.2
- new net OPOUTA: IC1.SO, R14.1
- new net SNSOUT: IC1.SNSOUT, U7A.PB2
- new net VCP: C9.2, IC1.VCP
- net !EMS: now also IC1.NSLEEP, U7A.PB11; no longer U3.ENA, U3.ENB, U7A.PA4
- net +3V3: now also C14.2, C15.2, C2.2, C23.2, C28.2, C3.2, C4.2, U$1.4; no longer C1.1, C11.1, C2.1, C25.1, C3.1, C33.1, C4.1, C5.1, IC3.VCC, R10.1, R6.2, R9.1, U$1.1
- net +5V: now also C19.2, C22.2, C6.1, C7.1, C8.1, D1.C, D2.A, L1.2, R2.2, TP8.TP, U2.VCC; no longer C10.1, C9.1, L1.1, R1.1, TP6.TP
- net BUTTON: now also U7A.PB4; no longer C29.1, U7A.PC13
- net CAN_H: now also J2.2, R8.2, U2.CANH; no longer IC3.CANH, J1.1, J1.MP1, R8.1
- net CAN_L: now also J2.1, R8.1, U2.CANL; no longer IC3.CANL, J1.2, J1.MP2, R8.2
- net CAN_RX: now also U2.RXD; no longer IC3.R
- net CAN_TX: now also U2.TXD; no longer IC3.D
- net ENC_A: now also U7A.PA15; no longer U7A.PA0
- net ENC_B: now also U7A.PB3; no longer U7A.PA1
- net FB: now also C8.2, R2.1, U1.FB; no longer IC2.FB, R2.2
- net GH1: now also IC1.GH1; no longer U3.GHA
- net GH2: now also IC1.GH2; no longer U3.GHB
- net GL1: now also IC1.GL1; no longer U3.GLA
- net GL2: now also IC1.GL2; no longer U3.GLB
- net GNDA: now also C1.1, C11.1, C15.1, C16.1, C17.1, C18.1, C19.1, C2.1, C21.2, C22.1, C23.1, C24.1, C27.1, C28.1, C3.1, C30.2, C31.2, C4.1, D1.A, IC1.GND_1, IC1.GND_2, IC1.GND_3, IC1.SN, R1.1, TP6.TP, U$1.1, U1.GND, U11.REF1, U2.GND, U2.S; no longer C1.2, C10.2, C11.2, C18.-, C19.2, C2.2, C25.2, C26.2, C27.2, C28.2, C3.2, C30.-, C33.2, C4.2, C9.2, IC2.GND, IC3.GND, IC3.RS, R13.2, R2.1, R5.1, U$1.4, U11.IN+2, U11.IN-2, U3.EPAD, U3.GND, U3.GND_2, U3.GND_3, Y1.GND_1, Y1.GND_2
- net ISENSEB: now also C17.2, U7A.PA3; no longer C26.1, ISENSE.TP, U7A.PB1
- net N$12: now also C25.2; no longer C22.2
- net N$13: now also C26.2; no longer C24.2
- net N$38: now also C44.2; no longer C23.2
- net N$39: now also C43.2; no longer C21.2
- net NFAULT: now also IC1.NFAULT, U7A.PB0; no longer R9.2, U3.NFAULT, U7A.PA3
- net OUT+: now also C43.1, IC1.SH2; no longer C15.1, C21.1, U3.SHB
- net OUT-: now also C44.1, IC1.SH1; no longer C16.2, C23.1, U3.SHA
- net SP: now also IC1.SP
- net TEMP: now also C16.2, U7A.PA7; no longer C27.1, U7A.PA6
- net VCC: now also C13.2, C21.1, C29.1, C30.1, C31.1, C5.1, C9.1, D2.C, IC1.VM, U1.EN/SS, U1.VIN; no longer C18.+, C19.1, C30.+, C6.1, C7.1, IC2.EN, IC2.VIN, U3.VIN
- net VCS: now also C25.1, C26.1; no longer C22.1, C24.1, U3.LSS
- net VREF: now also IC1.VREF; no longer U11.REF1
- net VSENSE: now also C1.2, U7A.PB1; no longer C28.1, U7A.PB0
Other:
- note removed: "U11 = INA2181A2 / 0.15 V/A / sat 19.9A"
- moved on the sheet: C1, C10, C11, C12, C13, C14, C15, C16, C17, C19, C2, C20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
